File: beacons/beaconboard3.sch (EAGLE design)
At the start: 42 parts, among them IC1 7805TV, Q1 2N3904, Q2 16MHz, Q3 2N3904, Q4 2N3904, Q5 2N3904

Commit message: Updated beaconboard with staff suggestions
Parts:
- added C7: 0.1uF, SparkFun-Passives:CAPPTH1
- added MODE3: SPD_SLIDE_SWITCH, e11:SPD_SLIDE_SWITCH
- added R16: 33, SparkFun-Resistors:RESISTORPTH-1/4W
- added U$6: FTDI, e11:FTDI
- R1: value 30 -> 33
- R11: value 200 -> 20k
- R13, R14, R15: value 55 -> 100
- R3: value 330 -> 10k
- renumbered PB1 to PUSH1, PB2 to PUSH2
Connections:
- new net DTR: C7.2, U$6.DTR
- new net MODE3: MODE3.2, U$4.PB1/OC1A/PCINT1
- new net N$25: LED2.C, R16.2
- new net RXI: U$4.PD0/PCINT16/RXD, U$6.TXO
- new net TXO: U$4.PD1/PCINT17/TXD, U$6.RXI
- net GND: now also MODE3.3, U$6.CTS, U$6.GND
- net N$1: now also R16.1
- net N$11: now also C7.1
- net N$3: no longer LED2.C
- net VCC: now also LED1.A, LED2.A, MODE3.1, R13.2, R14.2, R15.2, R3.2, U$6.VCC
- net VDD: no longer LED1.A, LED2.A, R13.2, R14.2, R15.2, R3.2
Other:
- moved on the sheet: R1
