File: beacons/v3/beaconboard3.sch (EAGLE design)
At the start: 46 parts, among them IC1 7805TV, Q1 2N3904, Q2 16MHz, Q3 2N3904, Q4 2N3904, Q5 2N3904

Commit message: Updated readme. Added omron switches in version 3
Parts:
- removed PUSH1, PUSH2: D6_PUSHBUTTON, e11:D6_PUSHBUTTON
- added S2, S3: (no value), switch-omron:40-XX
Connections:
- net BUMPER: now also S2.S, S2.S1, S3.S, S3.S1; no longer PUSH1.2, PUSH2.2
- net GND: now also S2.P, S2.P1, S3.P, S3.P1; no longer PUSH1.1, PUSH2.1
Changed lines of the file:
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@@
 <part name="VDD3" library="supply1" deviceset="VDD" device=""/>
 <part name="SUPPLY12" library="supply2" deviceset="GND" device=""/>
-<part name="PUSH1" library="e11" deviceset="D6_PUSHBUTTON" device=""/>
-<part name="PUSH2" library="e11" deviceset="D6_PUSHBUTTON" device=""/>
 <part name="U$2" library="e11" deviceset="BPW77NA" device=""/>
 <part name="SUPPLY13" library="supply2" deviceset="GND" device=""/>
@@
 <part name="R16" library="SparkFun-Resistors" deviceset="RESISTOR" device="PTH-1/4W" value="33"/>
 <part name="MODE3" library="e11" deviceset="SPD_SLIDE_SWITCH" device=""/>
+<part name="S2" library="switch-omron" deviceset="40-XX" device=""/>
+<part name="S3" library="switch-omron" deviceset="40-XX" device=""/>
 </parts>
 <sheets>
@@
 <instance part="VDD3" gate="G$1" x="-20.32" y="116.84"/>
 <instance part="SUPPLY12" gate="GND" x="-20.32" y="106.68"/>
-<instance part="PUSH1" gate="G$1" x="2.54" y="48.26" rot="R90"/>
-<instance part="PUSH2" gate="G$1" x="15.24" y="48.26" rot="R90"/>
 <instance part="U$2" gate="G$1" x="215.9" y="78.74"/>
 <instance part="SUPPLY13" gate="GND" x="218.44" y="71.12"/>
@@
 <instance part="R16" gate="G$1" x="195.58" y="116.84" rot="R90"/>
 <instance part="MODE3" gate="G$1" x="25.4" y="-20.32"/>
+<instance part="S2" gate="1" x="2.54" y="48.26"/>
+<instance part="S3" gate="1" x="12.7" y="48.26"/>
 </instances>
 <busses>
@@
 <segment>
 <wire x1="15.24" y1="43.18" x2="15.24" y2="35.56" width="0.1524" layer="91"/>
-<pinref part="PUSH1" gate="G$1" pin="1"/>
-<wire x1="2.54" y1="43.18" x2="15.24" y2="43.18" width="0.1524" layer="91"/>
+<wire x1="2.54" y1="43.18" x2="5.08" y2="43.18" width="0.1524" layer="91"/>
 <pinref part="SUPPLY11" gate="GND" pin="GND"/>
-<pinref part="PUSH2" gate="G$1" pin="1"/>
+<pinref part="S3" gate="1" pin="P"/>
+<wire x1="5.08" y1="43.18" x2="12.7" y2="43.18" width="0.1524" layer="91"/>
+<wire x1="12.7" y1="43.18" x2="15.24" y2="43.18" width="0.1524" layer="91"/>
+<junction x="12.7" y="43.18"/>
+<pinref part="S3" gate="1" pin="P1"/>
 <junction x="15.24" y="43.18"/>
+<pinref part="S2" gate="1" pin="P"/>
+<pinref part="S2" gate="1" pin="P1"/>
+<junction x="5.08" y="43.18"/>
 </segment>
 <segment>
@@
 <net name="BUMPER" class="0">
 <segment>
+<junction x="20.32" y="53.34"/>
 <wire x1="20.32" y1="53.34" x2="15.24" y2="53.34" width="0.1524" layer="91"/>
-<junction x="20.32" y="53.34"/>
-<wire x1="15.24" y1="53.34" x2="2.54" y2="53.34" width="0.1524" layer="91"/>
+<wire x1="15.24" y1="53.34" x2="12.7" y2="53.34" width="0.1524" layer="91"/>
+<wire x1="12.7" y1="53.34" x2="5.08" y2="53.34" width="0.1524" layer="91"/>
+<wire x1="5.08" y1="53.34" x2="2.54" y2="53.34" width="0.1524" layer="91"/>
 <wire x1="20.32" y1="53.34" x2="35.56" y2="53.34" width="0.1524" layer="91"/>
 <label x="35.56" y="53.34" size="1.778" layer="95"/>
-<pinref part="PUSH1" gate="G$1" pin="2"/>
 <pinref part="R11" gate="G$1" pin="2"/>
 <junction x="20.32" y="53.34"/>
-<pinref part="PUSH2" gate="G$1" pin="2"/>
+<pinref part="S3" gate="1" pin="S"/>
+<junction x="12.7" y="53.34"/>
+<pinref part="S3" gate="1" pin="S1"/>
 <junction x="15.24" y="53.34"/>
-</segment>
-<segment>
+<pinref part="S2" gate="1" pin="S"/>
+<pinref part="S2" gate="1" pin="S1"/>
+<junction x="5.08" y="53.34"/>
+</segment>
+<segment>

Commit message: Added pdf of sch and updated boms
Parts:
- removed S2: (no value), switch-omron:40-XX
- added B3F-4050: (no value), switch-omron:40-XX
- renumbered LED2 to HF5-R5590
Connections:
- net BUMPER: now also B3F-4050.S, B3F-4050.S1; no longer S2.S, S2.S1
- net GND: now also B3F-4050.P, B3F-4050.P1; no longer S2.P, S2.P1
Other:
- moved on the sheet: J1
Changed lines of the file:
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@@
 <part name="SUPPLY3" library="supply2" deviceset="GND" device=""/>
 <part name="LED1" library="led" deviceset="LED-2AC-" device="CP41B-WES"/>
-<part name="LED2" library="led" deviceset="LED-2AC-" device="CP41B-WES"/>
+<part name="HF5-R5590" library="led" deviceset="LED-2AC-" device="CP41B-WES"/>
 <part name="SUPPLY4" library="supply2" deviceset="GND" device=""/>
 <part name="R1" library="SparkFun-Resistors" deviceset="RESISTOR" device="PTH-1/4W" value="33"/>
@@
 <part name="R16" library="SparkFun-Resistors" deviceset="RESISTOR" device="PTH-1/4W" value="33"/>
 <part name="MODE3" library="e11" deviceset="SPD_SLIDE_SWITCH" device=""/>
-<part name="S2" library="switch-omron" deviceset="40-XX" device=""/>
+<part name="B3F-4050" library="switch-omron" deviceset="40-XX" device=""/>
 <part name="S3" library="switch-omron" deviceset="40-XX" device=""/>
 </parts>
@@
 <instance part="U$4" gate="G$1" x="124.46" y="-2.54"/>
 <instance part="Q1" gate="1" x="187.96" y="104.14"/>
-<instance part="J1" gate="G$1" x="-33.02" y="111.76"/>
+<instance part="J1" gate="G$1" x="93.98" y="137.16"/>
 <instance part="IC1" gate="A1" x="30.48" y="93.98"/>
 <instance part="C2" gate="G$1" x="12.7" y="91.44"/>
@@
 <instance part="SUPPLY3" gate="GND" x="182.88" y="35.56"/>
 <instance part="LED1" gate="G$1" x="185.42" y="129.54"/>
-<instance part="LED2" gate="G$1" x="195.58" y="129.54"/>
+<instance part="HF5-R5590" gate="G$1" x="195.58" y="129.54"/>
 <instance part="SUPPLY4" gate="GND" x="190.5" y="93.98"/>
 <instance part="R1" gate="G$1" x="185.42" y="116.84" rot="R90"/>
@@
 <instance part="V_OUT6" gate="1" x="20.32" y="66.04"/>
 <instance part="R11" gate="G$1" x="20.32" y="58.42" rot="R270"/>
-<instance part="VDD3" gate="G$1" x="-20.32" y="116.84"/>
-<instance part="SUPPLY12" gate="GND" x="-20.32" y="106.68"/>
+<instance part="VDD3" gate="G$1" x="106.68" y="142.24"/>
+<instance part="SUPPLY12" gate="GND" x="106.68" y="132.08"/>
 <instance part="U$2" gate="G$1" x="215.9" y="78.74"/>
 <instance part="SUPPLY13" gate="GND" x="218.44" y="71.12"/>
@@
 <instance part="R16" gate="G$1" x="195.58" y="116.84" rot="R90"/>
 <instance part="MODE3" gate="G$1" x="25.4" y="-20.32"/>
-<instance part="S2" gate="1" x="2.54" y="48.26"/>
+<instance part="B3F-4050" gate="1" x="0" y="48.26"/>
 <instance part="S3" gate="1" x="12.7" y="48.26"/>
 </instances>
@@
 <pinref part="J1" gate="G$1" pin="3"/>
 <pinref part="VDD3" gate="G$1" pin="VDD"/>
-<wire x1="-20.32" y1="114.3" x2="-27.94" y2="114.3" width="0.1524" layer="91"/>
+<wire x1="106.68" y1="139.7" x2="99.06" y2="139.7" width="0.1524" layer="91"/>
 </segment>
 </net>
@@
 <pinref part="LED1" gate="G$1" pin="A"/>
 <wire x1="185.42" y1="134.62" x2="185.42" y2="132.08" width="0.1524" layer="91"/>
-<pinref part="LED2" gate="G$1" pin="A"/>
+<pinref part="HF5-R5590" gate="G$1" pin="A"/>
 <wire x1="190.5" y1="134.62" x2="195.58" y2="134.62" width="0.1524" layer="91"/>
 <wire x1="195.58" y1="134.62" x2="195.58" y2="132.08" width="0.1524" layer="91"/>
@@
 <pinref part="J1" gate="G$1" pin="1"/>
 <pinref part="SUPPLY12" gate="GND" pin="GND"/>
-<wire x1="-20.32" y1="109.22" x2="-27.94" y2="109.22" width="0.1524" layer="91"/>
+<wire x1="106.68" y1="134.62" x2="99.06" y2="134.62" width="0.1524" layer="91"/>
 </segment>
 <segment>
 <wire x1="15.24" y1="43.18" x2="15.24" y2="35.56" width="0.1524" layer="91"/>
-<wire x1="2.54" y1="43.18" x2="5.08" y2="43.18" width="0.1524" layer="91"/>
+<wire x1="0" y1="43.18" x2="2.54" y2="43.18" width="0.1524" layer="91"/>
 <pinref part="SUPPLY11" gate="GND" pin="GND"/>
 <pinref part="S3" gate="1" pin="P"/>
-<wire x1="5.08" y1="43.18" x2="12.7" y2="43.18" width="0.1524" layer="91"/>
+<wire x1="2.54" y1="43.18" x2="12.7" y2="43.18" width="0.1524" layer="91"/>
 <wire x1="12.7" y1="43.18" x2="15.24" y2="43.18" width="0.1524" layer="91"/>
 <junction x="12.7" y="43.18"/>
 <pinref part="S3" gate="1" pin="P1"/>
 <junction x="15.24" y="43.18"/>
-<pinref part="S2" gate="1" pin="P"/>
-<pinref part="S2" gate="1" pin="P1"/>
-<junction x="5.08" y="43.18"/>
+<pinref part="B3F-4050" gate="1" pin="P"/>
+<pinref part="B3F-4050" gate="1" pin="P1"/>
+<junction x="2.54" y="43.18"/>
 </segment>
 <segment>
@@
 <wire x1="20.32" y1="53.34" x2="15.24" y2="53.34" width="0.1524" layer="91"/>
 <wire x1="15.24" y1="53.34" x2="12.7" y2="53.34" width="0.1524" layer="91"/>
-<wire x1="12.7" y1="53.34" x2="5.08" y2="53.34" width="0.1524" layer="91"/>
-<wire x1="5.08" y1="53.34" x2="2.54" y2="53.34" width="0.1524" layer="91"/>
+<wire x1="12.7" y1="53.34" x2="2.54" y2="53.34" width="0.1524" layer="91"/>
+<wire x1="2.54" y1="53.34" x2="0" y2="53.34" width="0.1524" layer="91"/>
 <wire x1="20.32" y1="53.34" x2="35.56" y2="53.34" width="0.1524" layer="91"/>
 <label x="35.56" y="53.34" size="1.778" layer="95"/>
@@
 <pinref part="S3" gate="1" pin="S1"/>
 <junction x="15.24" y="53.34"/>
-<pinref part="S2" gate="1" pin="S"/>
-<pinref part="S2" gate="1" pin="S1"/>
-<junction x="5.08" y="53.34"/>
+<pinref part="B3F-4050" gate="1" pin="S"/>
+<pinref part="B3F-4050" gate="1" pin="S1"/>
+<junction x="2.54" y="53.34"/>
 </segment>
 <segment>
@@
 <segment>
 <pinref part="R16" gate="G$1" pin="2"/>
-<pinref part="LED2" gate="G$1" pin="C"/>
+<pinref part="HF5-R5590" gate="G$1" pin="C"/>
 <wire x1="195.58" y1="121.92" x2="195.58" y2="124.46" width="0.1524" layer="91"/>
 </segment>
